File: KiCad/motor_driver.sch (KiCad schematic (older format))
At the start: 18 parts

Commit message: adding altium docs
Parts:
- added P?: USB_OTG, symbol USB_OTG
Connections:
- net labels added: SWITCHER?, USB_D+, USB_D-
- wire segments 58 -> 63
- no-connect marks 0 -> 1
Other:
- note added: "+3.3V Power"
- note added: "Debug Header"
- note added: "H-Bridge A"
- note added: "H-Bridge B"
- note added: "Micro - ATXMEGA32C4"
- note added: "Pick switcher vs LDO\nPick 2 diodes\nPick Cap for bootstrap\nPick Battery - should be flexible for higher motor power?\nPick motor control method? Encoder option?\nCheck out Crowdsupply motor driver schematics\nBreakout for ultrasonic sensor??"
- note added: "USB & Power Connector"
- moved on the sheet: C?, D?, IC?, Q?, R?
